File: DP65_PCB/DP65.kicad_sch (KiCad schematic)
At the start: 148 parts, among them J1 Conn_01x02, J2 Conn_01x02

Commit message: commit
Parts:
- removed C1, C2, C3, C4: 10nF, symbol Device:C_Small
- removed D101, D102: D_Small, Diode_SMD:D_SOD-123, symbol Device:D_Small
- removed Display1: nice!view, nice_view:nice_view, symbol nice_view:nice!view
- removed ENC1: ENC_L, symbol Device:RotaryEncoder_Switch
- removed ENC2: ENC_R, symbol Device:RotaryEncoder_Switch
- added C5, C6, C7, C8: 100nF, Capacitor_SMD:C_0805_2012Metric_Pad1.18x1.45mm_HandSolder, symbol Device:C_Small
- added Display_LEFT1: nice!view, Connector_PinHeader_2.54mm:PinHeader_1x05_P2.54mm_Vertical, symbol nice_view:nice!view
- added ENC_LEFT1, ENC_RIGHT1: AS5600, AS5600:SOIC8, symbol AS5600:AS5600
- added R1, R2, R3, R4: 10k, Resistor_SMD:R_0805_2012Metric, symbol Device:R
- BAT_SW_L1: renamed from BAT_SW_L; footprint (none) -> Button_Switch_THT:SW_Slide_SPDT_Angled_CK_OS102011MA1Q; LCSC (none) -> C221530
- BAT_SW_R1: renamed from BAT_SW_R; footprint (none) -> Button_Switch_THT:SW_Slide_SPDT_Angled_CK_OS102011MA1Q; LCSC (none) -> C221530
- D1, D10, D11, D12, D13, D14, D15, D16, D17, D18, D19, D2, D20, D21, D22, D23, D24, D25, D26, D27, D28, D29, D3, D30, D31, D32, D33, D34, D35, D36, D37, D38, D39, D4, D40, D41, D42, D43, D44, D45, D46, D47, D48, D49, D5, D50, D51, D52, D53, D54, D55, D56, D57, D58, D59, D6, D60, D61, D62, D63, D64, D65, D7, D8, D9: LCSC (none) -> C81598
- Display_RIGHT1: renamed from Display2; footprint nice_view:nice_view -> Connector_PinHeader_2.54mm:PinHeader_1x05_P2.54mm_Vertical
- J1, J2: footprint Connector_JST:JST_PH_B2B-PH-SM4-TB_1x02-1MP_P2.00mm_Vertical -> Connector_JST:JST_PH_S2B-PH-SM4-TB_1x02-1MP_P2.00mm_Horizontal; LCSC (none) -> C295747
- K_0, K_1, K_2, K_3, K_4, K_5, K_6, K_7, K_8, K_9: footprint PCM_marbastlib-choc:SW_choc_v1_HS_CPG135001S30_1u -> PCM_Switch_Keyboard_Hotswap_Kailh:SW_Hotswap_Kailh_Choc_V1V2_1.00u; LCSC (none) -> C5333465
- K_A1: renamed from K_A; footprint PCM_marbastlib-choc:SW_choc_v1_HS_CPG135001S30_1u -> PCM_Switch_Keyboard_Hotswap_Kailh:SW_Hotswap_Kailh_Choc_V1V2_1.00u; LCSC (none) -> C5333465
- K_ALT_L1: renamed from K_ALT_L; footprint PCM_marbastlib-choc:SW_choc_v1_HS_CPG135001S30_1u -> PCM_Switch_Keyboard_Hotswap_Kailh:SW_Hotswap_Kailh_Choc_V1V2_1.25u; LCSC (none) -> C5333465
- K_ALT_R1: renamed from K_ALT_R; footprint PCM_marbastlib-choc:SW_choc_v1_HS_CPG135001S30_1u -> PCM_Switch_Keyboard_Hotswap_Kailh:SW_Hotswap_Kailh_Choc_V1V2_1.25u; LCSC (none) -> C5333465
- K_B1: renamed from K_B; footprint PCM_marbastlib-choc:SW_choc_v1_HS_CPG135001S30_1u -> PCM_Switch_Keyboard_Hotswap_Kailh:SW_Hotswap_Kailh_Choc_V1V2_1.00u; LCSC (none) -> C5333465
- K_BACKSPACE1: renamed from K_BACKSPACE; footprint PCM_marbastlib-choc:SW_choc_v1_HS_CPG135001S30_1u -> PCM_Switch_Keyboard_Hotswap_Kailh:SW_Hotswap_Kailh_Choc_V1V2_2.00u; LCSC (none) -> C5333465
- K_C1: renamed from K_C; footprint PCM_marbastlib-choc:SW_choc_v1_HS_CPG135001S30_1u -> PCM_Switch_Keyboard_Hotswap_Kailh:SW_Hotswap_Kailh_Choc_V1V2_1.00u; LCSC (none) -> C5333465
- K_CAPS1: renamed from K_CAPS; footprint PCM_marbastlib-choc:SW_choc_v1_HS_CPG135001S30_1u -> PCM_Switch_Keyboard_Hotswap_Kailh:SW_Hotswap_Kailh_Choc_V1V2_1.75u; LCSC (none) -> C5333465
- K_COMMA1: renamed from K_COMMA; footprint PCM_marbastlib-choc:SW_choc_v1_HS_CPG135001S30_1u -> PCM_Switch_Keyboard_Hotswap_Kailh:SW_Hotswap_Kailh_Choc_V1V2_1.00u; LCSC (none) -> C5333465
- K_CRTL1: renamed from K_CRTL; footprint PCM_marbastlib-choc:SW_choc_v1_HS_CPG135001S30_1u -> PCM_Switch_Keyboard_Hotswap_Kailh:SW_Hotswap_Kailh_Choc_V1V2_1.25u; LCSC (none) -> C5333465
- K_D1: renamed from K_D; footprint PCM_marbastlib-choc:SW_choc_v1_HS_CPG135001S30_1u -> PCM_Switch_Keyboard_Hotswap_Kailh:SW_Hotswap_Kailh_Choc_V1V2_1.00u; LCSC (none) -> C5333465
- K_DOWN_ARR1: renamed from K_DOWN_ARR; footprint PCM_marbastlib-choc:SW_choc_v1_HS_CPG135001S30_1u -> PCM_Switch_Keyboard_Hotswap_Kailh:SW_Hotswap_Kailh_Choc_V1V2_1.00u; LCSC (none) -> C5333465
- K_E1: renamed from K_E; footprint PCM_marbastlib-choc:SW_choc_v1_HS_CPG135001S30_1u -> PCM_Switch_Keyboard_Hotswap_Kailh:SW_Hotswap_Kailh_Choc_V1V2_1.00u; LCSC (none) -> C5333465
- K_ENTER1: renamed from K_ENTER; footprint PCM_marbastlib-choc:SW_choc_v1_HS_CPG135001S30_1u -> PCM_Switch_Keyboard_Hotswap_Kailh:SW_Hotswap_Kailh_Choc_V1V2_2.25u; LCSC (none) -> C5333465
- K_ESC1: renamed from K_ESC; footprint PCM_marbastlib-choc:SW_choc_v1_HS_CPG135001S30_1u -> PCM_Switch_Keyboard_Hotswap_Kailh:SW_Hotswap_Kailh_Choc_V1V2_1.00u; LCSC (none) -> C5333465
- K_F1: renamed from K_F; footprint PCM_marbastlib-choc:SW_choc_v1_HS_CPG135001S30_1u -> PCM_Switch_Keyboard_Hotswap_Kailh:SW_Hotswap_Kailh_Choc_V1V2_1.00u; LCSC (none) -> C5333465
- K_FN1, K_FN2: footprint PCM_marbastlib-choc:SW_choc_v1_HS_CPG135001S30_1u -> PCM_Switch_Keyboard_Hotswap_Kailh:SW_Hotswap_Kailh_Choc_V1V2_1.25u; LCSC (none) -> C5333465
- K_G1: renamed from K_G; footprint PCM_marbastlib-choc:SW_choc_v1_HS_CPG135001S30_1u -> PCM_Switch_Keyboard_Hotswap_Kailh:SW_Hotswap_Kailh_Choc_V1V2_1.00u; LCSC (none) -> C5333465
- K_H1: renamed from K_H; footprint PCM_marbastlib-choc:SW_choc_v1_HS_CPG135001S30_1u -> PCM_Switch_Keyboard_Hotswap_Kailh:SW_Hotswap_Kailh_Choc_V1V2_1.00u; LCSC (none) -> C5333465
- K_I1: renamed from K_I; footprint PCM_marbastlib-choc:SW_choc_v1_HS_CPG135001S30_1u -> PCM_Switch_Keyboard_Hotswap_Kailh:SW_Hotswap_Kailh_Choc_V1V2_1.00u; LCSC (none) -> C5333465
- K_J1: renamed from K_J; footprint PCM_marbastlib-choc:SW_choc_v1_HS_CPG135001S30_1u -> PCM_Switch_Keyboard_Hotswap_Kailh:SW_Hotswap_Kailh_Choc_V1V2_1.00u; LCSC (none) -> C5333465
- K_K1: renamed from K_K; footprint PCM_marbastlib-choc:SW_choc_v1_HS_CPG135001S30_1u -> PCM_Switch_Keyboard_Hotswap_Kailh:SW_Hotswap_Kailh_Choc_V1V2_1.00u; LCSC (none) -> C5333465
- K_L1: renamed from K_L; footprint PCM_marbastlib-choc:SW_choc_v1_HS_CPG135001S30_1u -> PCM_Switch_Keyboard_Hotswap_Kailh:SW_Hotswap_Kailh_Choc_V1V2_1.00u; LCSC (none) -> C5333465
- K_LEFT_ARR1: renamed from K_LEFT_ARR; footprint PCM_marbastlib-choc:SW_choc_v1_HS_CPG135001S30_1u -> PCM_Switch_Keyboard_Hotswap_Kailh:SW_Hotswap_Kailh_Choc_V1V2_1.00u; LCSC (none) -> C5333465
- K_L_BRAC1: renamed from K_L_BRAC; footprint PCM_marbastlib-choc:SW_choc_v1_HS_CPG135001S30_1u -> PCM_Switch_Keyboard_Hotswap_Kailh:SW_Hotswap_Kailh_Choc_V1V2_1.00u; LCSC (none) -> C5333465
- K_M1: renamed from K_M; footprint PCM_marbastlib-choc:SW_choc_v1_HS_CPG135001S30_1u -> PCM_Switch_Keyboard_Hotswap_Kailh:SW_Hotswap_Kailh_Choc_V1V2_1.00u; LCSC (none) -> C5333465
- K_MINUS1: renamed from K_MINUS; footprint PCM_marbastlib-choc:SW_choc_v1_HS_CPG135001S30_1u -> PCM_Switch_Keyboard_Hotswap_Kailh:SW_Hotswap_Kailh_Choc_V1V2_1.00u; LCSC (none) -> C5333465
- K_N1: renamed from K_N; footprint PCM_marbastlib-choc:SW_choc_v1_HS_CPG135001S30_1u -> PCM_Switch_Keyboard_Hotswap_Kailh:SW_Hotswap_Kailh_Choc_V1V2_1.00u; LCSC (none) -> C5333465
- K_O1: renamed from K_O; footprint PCM_marbastlib-choc:SW_choc_v1_HS_CPG135001S30_1u -> PCM_Switch_Keyboard_Hotswap_Kailh:SW_Hotswap_Kailh_Choc_V1V2_1.00u; LCSC (none) -> C5333465
- K_P1: renamed from K_P; footprint PCM_marbastlib-choc:SW_choc_v1_HS_CPG135001S30_1u -> PCM_Switch_Keyboard_Hotswap_Kailh:SW_Hotswap_Kailh_Choc_V1V2_1.00u; LCSC (none) -> C5333465
- K_PERIOD1: renamed from K_PERIOD; footprint PCM_marbastlib-choc:SW_choc_v1_HS_CPG135001S30_1u -> PCM_Switch_Keyboard_Hotswap_Kailh:SW_Hotswap_Kailh_Choc_V1V2_1.00u; LCSC (none) -> C5333465
- K_PIPE1: renamed from K_PIPE; footprint PCM_marbastlib-choc:SW_choc_v1_HS_CPG135001S30_1u -> PCM_Switch_Keyboard_Hotswap_Kailh:SW_Hotswap_Kailh_Choc_V1V2_1.50u; LCSC (none) -> C5333465
- K_PLUS1: renamed from K_PLUS; footprint PCM_marbastlib-choc:SW_choc_v1_HS_CPG135001S30_1u -> PCM_Switch_Keyboard_Hotswap_Kailh:SW_Hotswap_Kailh_Choc_V1V2_1.00u; LCSC (none) -> C5333465
- K_Q1: renamed from K_Q; footprint PCM_marbastlib-choc:SW_choc_v1_HS_CPG135001S30_1u -> PCM_Switch_Keyboard_Hotswap_Kailh:SW_Hotswap_Kailh_Choc_V1V2_1.00u; LCSC (none) -> C5333465
- K_QUOTE1: renamed from K_QUOTE; footprint PCM_marbastlib-choc:SW_choc_v1_HS_CPG135001S30_1u -> PCM_Switch_Keyboard_Hotswap_Kailh:SW_Hotswap_Kailh_Choc_V1V2_1.00u; LCSC (none) -> C5333465
- K_R1: renamed from K_R; footprint PCM_marbastlib-choc:SW_choc_v1_HS_CPG135001S30_1u -> PCM_Switch_Keyboard_Hotswap_Kailh:SW_Hotswap_Kailh_Choc_V1V2_1.00u; LCSC (none) -> C5333465
- K_RIGHT_ARR1: renamed from K_RIGHT_ARR; footprint PCM_marbastlib-choc:SW_choc_v1_HS_CPG135001S30_1u -> PCM_Switch_Keyboard_Hotswap_Kailh:SW_Hotswap_Kailh_Choc_V1V2_1.00u; LCSC (none) -> C5333465
- K_R_BRAC1: renamed from K_R_BRAC; footprint PCM_marbastlib-choc:SW_choc_v1_HS_CPG135001S30_1u -> PCM_Switch_Keyboard_Hotswap_Kailh:SW_Hotswap_Kailh_Choc_V1V2_1.00u; LCSC (none) -> C5333465
- K_S1: renamed from K_S; footprint PCM_marbastlib-choc:SW_choc_v1_HS_CPG135001S30_1u -> PCM_Switch_Keyboard_Hotswap_Kailh:SW_Hotswap_Kailh_Choc_V1V2_1.00u; LCSC (none) -> C5333465
- K_SEMICOLON1: renamed from K_SEMICOLON; footprint PCM_marbastlib-choc:SW_choc_v1_HS_CPG135001S30_1u -> PCM_Switch_Keyboard_Hotswap_Kailh:SW_Hotswap_Kailh_Choc_V1V2_1.00u; LCSC (none) -> C5333465
- K_SHIFT1: renamed from K_SHIFT; footprint PCM_marbastlib-choc:SW_choc_v1_HS_CPG135001S30_1u -> PCM_Switch_Keyboard_Hotswap_Kailh:SW_Hotswap_Kailh_Choc_V1V2_2.25u; LCSC (none) -> C5333465
- K_SHIFT2: renamed from K_SHIFT; footprint PCM_marbastlib-choc:SW_choc_v1_HS_CPG135001S30_1u -> PCM_Switch_Keyboard_Hotswap_Kailh:SW_Hotswap_Kailh_Choc_V1V2_1.75u; LCSC (none) -> C5333465
- K_SLASH1: renamed from K_SLASH; footprint PCM_marbastlib-choc:SW_choc_v1_HS_CPG135001S30_1u -> PCM_Switch_Keyboard_Hotswap_Kailh:SW_Hotswap_Kailh_Choc_V1V2_1.00u; LCSC (none) -> C5333465
- K_SPACE_L1: renamed from K_SPACE_L; footprint PCM_marbastlib-choc:SW_choc_v1_HS_CPG135001S30_1u -> PCM_Switch_Keyboard_Hotswap_Kailh:SW_Hotswap_Kailh_Choc_V1V2_2.25u; LCSC (none) -> C5333465
- K_SPACE_R1: renamed from K_SPACE_R; footprint PCM_marbastlib-choc:SW_choc_v1_HS_CPG135001S30_1u -> PCM_Switch_Keyboard_Hotswap_Kailh:SW_Hotswap_Kailh_Choc_V1V2_2.25u; LCSC (none) -> C5333465
- K_T1: renamed from K_T; footprint PCM_marbastlib-choc:SW_choc_v1_HS_CPG135001S30_1u -> PCM_Switch_Keyboard_Hotswap_Kailh:SW_Hotswap_Kailh_Choc_V1V2_1.00u; LCSC (none) -> C5333465
- K_TAB1: renamed from K_TAB; footprint PCM_marbastlib-choc:SW_choc_v1_HS_CPG135001S30_1u -> PCM_Switch_Keyboard_Hotswap_Kailh:SW_Hotswap_Kailh_Choc_V1V2_1.50u; LCSC (none) -> C5333465
- K_U1: renamed from K_U; footprint PCM_marbastlib-choc:SW_choc_v1_HS_CPG135001S30_1u -> PCM_Switch_Keyboard_Hotswap_Kailh:SW_Hotswap_Kailh_Choc_V1V2_1.00u; LCSC (none) -> C5333465
- K_UP_ARR1: renamed from K_UP_ARR; footprint PCM_marbastlib-choc:SW_choc_v1_HS_CPG135001S30_1u -> PCM_Switch_Keyboard_Hotswap_Kailh:SW_Hotswap_Kailh_Choc_V1V2_1.00u; LCSC (none) -> C5333465
- K_V1: renamed from K_V; footprint PCM_marbastlib-choc:SW_choc_v1_HS_CPG135001S30_1u -> PCM_Switch_Keyboard_Hotswap_Kailh:SW_Hotswap_Kailh_Choc_V1V2_1.00u; LCSC (none) -> C5333465
- K_W1: renamed from K_W; footprint PCM_marbastlib-choc:SW_choc_v1_HS_CPG135001S30_1u -> PCM_Switch_Keyboard_Hotswap_Kailh:SW_Hotswap_Kailh_Choc_V1V2_1.00u; LCSC (none) -> C5333465
- K_WIN1: renamed from K_WIN; footprint PCM_marbastlib-choc:SW_choc_v1_HS_CPG135001S30_1u -> PCM_Switch_Keyboard_Hotswap_Kailh:SW_Hotswap_Kailh_Choc_V1V2_1.25u; LCSC (none) -> C5333465
- K_X1: renamed from K_X; footprint PCM_marbastlib-choc:SW_choc_v1_HS_CPG135001S30_1u -> PCM_Switch_Keyboard_Hotswap_Kailh:SW_Hotswap_Kailh_Choc_V1V2_1.00u; LCSC (none) -> C5333465
- K_Y1: renamed from K_Y; footprint PCM_marbastlib-choc:SW_choc_v1_HS_CPG135001S30_1u -> PCM_Switch_Keyboard_Hotswap_Kailh:SW_Hotswap_Kailh_Choc_V1V2_1.00u; LCSC (none) -> C5333465
- K_Z1: renamed from K_Z; footprint PCM_marbastlib-choc:SW_choc_v1_HS_CPG135001S30_1u -> PCM_Switch_Keyboard_Hotswap_Kailh:SW_Hotswap_Kailh_Choc_V1V2_1.00u; LCSC (none) -> C5333465
- RST_SW1: renamed from RST_SW; footprint (none) -> Button_Switch_THT:SW_Tactile_SKHH_Angled; LCSC (none) -> C383800
- RST_SW2: footprint (none) -> Button_Switch_THT:SW_Tactile_SKHH_Angled; LCSC (none) -> C383800
- renumbered U_LEFT to NANO_LEFT1, U_RIGHT to NANO_RIGHT1
Connections:
- net L_CS: now also Display_LEFT1.5 (CS)
- net L_MOSI: now also Display_LEFT1.1 (MOSI)
- net L_ROW3: now also NANO_LEFT1.7 (P0.22); no longer NANO_LEFT1.25 (P1.01-LF)
- net L_ROW4: now also NANO_LEFT1.8 (P0.24); no longer NANO_LEFT1.26 (P1.02-LF)
- net L_SCK: now also Display_LEFT1.2 (SCK)
- net R_COL6: no longer K_FN2.1, K_H1.1, K_M1.1, K_Y1.1, NANO_RIGHT1.22 (P1.11-LF)
- net R_ROW2: now also NANO_RIGHT1.2 (P0.08); no longer NANO_RIGHT1.25 (P1.01-LF)
- net R_ROW3: now also NANO_RIGHT1.7 (P0.22); no longer NANO_RIGHT1.26 (P1.02-LF)
- net R_ROW4: now also NANO_RIGHT1.8 (P0.24); no longer NANO_RIGHT1.27 (P1.07-LF)
- net +3.3V renamed v3.3_RIGHT
- net v3.3_RIGHT: now also C7.2, C8.2, ENC_RIGHT1.1 (VDD5V), ENC_RIGHT1.2 (VDD3V3), R3.2, R4.2; no longer NANO_LEFT1.16 (3V3)
- net GND renamed GND_RIGHT
- net GND_RIGHT: now also C7.1, C8.1, ENC_RIGHT1.4 (GND), ENC_RIGHT1.8 (DIR); no longer J1.2 (Pin_2), NANO_LEFT1.14 (GND), NANO_LEFT1.28 (GND), NANO_LEFT1.3 (GND), NANO_LEFT1.4 (GND), RST_SW1.2
- net L_ENC_A renamed L_SCL
- net L_SCL: now also ENC_LEFT1.7 (SCL), R2.1
- net L_ENC_B renamed L_SDA
- net L_SDA: now also ENC_LEFT1.6 (SDA), R1.1
- net R_ENC_A renamed R_SCL
- net R_SCL: now also ENC_RIGHT1.7 (SCL), R4.1
- net R_ENC_B renamed R_SDA
- net R_SDA: now also ENC_RIGHT1.6 (SDA), R3.1
- new net GND_LEFT: C5.1, C6.1, Display_LEFT1.4 (GND), ENC_LEFT1.4 (GND), ENC_LEFT1.8 (DIR), J1.2 (Pin_2), NANO_LEFT1.14 (GND), NANO_LEFT1.28 (GND), NANO_LEFT1.3 (GND), NANO_LEFT1.4 (GND), RST_SW1.2
- new net R_COL7: K_FN2.1, K_H1.1, K_M1.1, K_Y1.1, NANO_RIGHT1.22 (P1.11-LF)
- new net v3.3_LEFT: C5.2, C6.2, Display_LEFT1.3 (VCC), ENC_LEFT1.1 (VDD5V), ENC_LEFT1.2 (VDD3V3), NANO_LEFT1.16 (3V3), R1.2, R2.2
- no-connect marks 7 -> 11
Other:
- note added: "LEFT SIDE"
- note added: "RIGHT SIDE"
- moved on the sheet: BAT_SW_L1, BAT_SW_R1, D1, D10, D11, D12, D13, D14, D15, D16, D17, D18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
